File: USB-C.kicad_pcb (KiCad board)
At the start: 4 copper layers, 30 x 20 mm, 5 parts, among them J1 USB_C_Receptacle, U18 USBLC6-2P6

Commit message: Demoday
Parts:
- removed U18: USBLC6-2P6, Package_TO_SOT_SMD:SOT-666
- added R1: 5k1, Resistor_SMD:R_0402_1005Metric, F.Cu at (129.4, 114.4)
- added R2: 5k1, Resistor_SMD:R_0402_1005Metric, F.Cu at (129.4, 116.4)
- added U1: USBLC6-2P6, Package_TO_SOT_SMD:SOT-666, F.Cu at (149.9, 108.1)
- added U2: ESP32-S3-WROOM-1, RF_Module:ESP32-S3-WROOM-1, F.Cu at (134.6, 96.7)
- F1: moved to F.Cu
- R3, R4: value 5k1 -> 22
- moved F1 35.5 mm to (114.9, 111.2), turned to 0 degrees
- moved R3 1.50 mm to (149.5, 110.6), turned to 90 degrees
- moved R4 1.31 mm to (150.5, 110.6)
Connections:
- R3 pad 1: GND -> Net-(J1-D--PadA7)
- R3 pad 2: Net-(J1-CC1) -> /D-
- R4 pad 1: GND -> /D+
- R4 pad 2: Net-(J1-CC2) -> Net-(J1-D+-PadA6)
Routing:
- net USB_D_P: track 2.06 -> 7.43 mm, vias 0 -> 2
- net USB_D_N: track 2.05 -> 6.80 mm, vias 0 -> 2
- net Net-(F1-Pad2): track 4.45 -> 0.00 mm, vias 4 -> 0
- net /D-: track 0.00 -> 3.61 mm
- net GND: track 3.29 -> 0.00 mm, vias 5 -> 4
- net /D+: track 0.00 -> 2.99 mm
- net Net-(J1-CC1): track 2.48 -> 0.00 mm
- net Net-(J1-D--PadA7): track 5.71 -> 3.89 mm, vias 2 -> 0
- net Net-(J1-D+-PadA6): track 5.56 -> 4.81 mm, vias 2 -> 0
- net Net-(J1-CC2): track 2.27 -> 1.78 mm, vias 0 -> 1
- net +5V: vias 5 -> 0
- added copper zone on In2.Cu, net GND
- removed copper zone on B.Cu, net +5V
- removed copper zone on In2.Cu, net +5V
- removed copper zone on B.Cu, net Net-(F1-Pad2)
Other:
- board text added: "LayerStack (JLCPCB) JLC04161H-3313"
