File: USB-C.kicad_sch (KiCad schematic)
At the start: 5 parts, among them J1 USB_C_Receptacle, U1 USBLC6-2P6

Commit message: Demoday
Parts:
- added R3, R4: 22, Resistor_SMD:R_0402_1005Metric, symbol Device:R
- added U2: ESP32-S3-WROOM-1, RF_Module:ESP32-S3-WROOM-1, symbol RF_Module:ESP32-S3-WROOM-1
Connections:
- net USB_D_N: now also U2.13 (USB_D-)
- net USB_D_P: now also U2.14 (USB_D+)
- net at J1.A6 (D+), J1.B6 (D+): now also R4.2; no longer U1.4 (I/O2)
- net at J1.A7 (D-), J1.B7 (D-): now also R3.1; no longer U1.6 (I/O1)
- new net: U2.1 (GND), U2.40 (GND), U2.41 (GND)
- new net D+: R4.1, U1.4 (I/O2)
- new net D-: R3.2, U1.6 (I/O1)
